File: KiCad/KiCad.kicad_pcb (KiCad board)
At the start: 2 copper layers, 45 x 65 mm, 31 parts, among them J1 3.7v, J2 writer, J3 SSD1306, J4 Micro_SD_Card_DW3AT-SF-PFJM5, J5 MotorA, J6 MotorB, J7 SPI, M1 SG90, M2 SG90, U1 NJM2845DL1-33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

Commit message: 修正
Parts:
- removed REF** (x4): MountingHole_2.2mm_M2, MountingHole:MountingHole_2.2mm_M2
- C6: value C_1608 -> 0.1μ
- R2: value R_1608 -> 10k
Connections:
- M1 pad 2: +3.3V -> 3.7v
- M2 pad 2: +3.3V -> 3.7v
Routing:
- net /IO18: track 6.44 -> 42.6 mm, vias 0 -> 2
- net /IO16: track 3.10 -> 30.3 mm, vias 0 -> 2
- net Net-(U2-IO5): track 0.00 -> 26.3 mm, vias 0 -> 2
- net +3.3V: track 148.7 -> 122.6 mm
- net 3.7v: track 22.6 -> 40.7 mm
- net Net-(J5-Pin_2): track 23.2 -> 21.6 mm
- net Net-(J5-Pin_1): track 16.8 -> 15.8 mm
- net GND: track 3.00 -> 3.80 mm, vias 0 -> 4
