File: KiCad/KiCad.kicad_sch (KiCad schematic)
At the start: 27 parts, among them J1 3.7v, J2 writer, J3 SSD1306, J4 Micro_SD_Card_DW3AT-SF-PFJM5, J5 MotorA, J6 MotorB, J7 SPI, M1 SG90, M2 SG90, U1 NJM2845DL1-33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

Commit message: 修正
Parts:
- added R10, R11, R12, R6, R7, R8, R9: 10k, Resistor_SMD:R_0603_1608Metric_Pad0.98x0.95mm_HandSolder, symbol MyLibrary:R_1608
Connections:
- net +3.3V: now also R12.1; no longer M1.2 (+), M2.2 (+)
- net 3.7v: now also M1.2 (+), M2.2 (+)
- net GND: now also R10.2, R11.2, R6.2, R7.2, R8.2, R9.2
- net IO12: now also R6.1
- net IO13: now also R7.1
- net IO14: now also R8.1
- net IO15: now also R9.1
- net IO32: now also R10.1
- net IO33: now also R11.1
- net at C7.1, S2.2, U2.24 (IO2): now also R12.2
